File: ItsyBitsy Display Add-On.sch (EAGLE design)
At the start: 15 parts, among them IC1 APX803, SW1 SPST_TACT-KMR2

Commit message: Fixed No ground to OLED, added names
Connections:
- net N$1 renamed C2P
- net N$2 renamed C2N
- net N$3 renamed C1P
- net N$4 renamed C1N
- net N$5 renamed VCOMH
- net N$6 renamed VCC
- net N$7 renamed IREF
Changed lines of the file:
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@@
 </segment>
 </net>
-<net name="N$1" class="0">
+<net name="C2P" class="0">
 <segment>
 <wire x1="78.74" y1="78.74" x2="76.2" y2="78.74" width="0.1524" layer="91"/>
@@
 </segment>
 </net>
-<net name="N$2" class="0">
+<net name="C2N" class="0">
 <segment>
 <wire x1="68.58" y1="78.74" x2="60.96" y2="78.74" width="0.1524" layer="91"/>
@@
 </segment>
 </net>
-<net name="N$3" class="0">
+<net name="C1P" class="0">
 <segment>
 <wire x1="78.74" y1="73.66" x2="71.12" y2="73.66" width="0.1524" layer="91"/>
@@
 </segment>
 </net>
-<net name="N$4" class="0">
+<net name="C1N" class="0">
 <segment>
 <wire x1="63.5" y1="73.66" x2="60.96" y2="73.66" width="0.1524" layer="91"/>
@@
 </segment>
 </net>
-<net name="N$5" class="0">
+<net name="VCOMH" class="0">
 <segment>
 <wire x1="78.74" y1="48.26" x2="53.34" y2="48.26" width="0.1524" layer="91"/>
@@
 </segment>
 </net>
-<net name="N$7" class="0">
+<net name="IREF" class="0">
 <segment>
 <wire x1="78.74" y1="50.8" x2="63.5" y2="50.8" width="0.1524" layer="91"/>
@@
 </segment>
 </net>
-<net name="N$6" class="0">
+<net name="VCC" class="0">
 <segment>
 <wire x1="78.74" y1="45.72" x2="48.26" y2="45.72" width="0.1524" layer="91"/>
